Commit message: feat: added camera joint to URDF

File: parcbot_description/urdf/parcbot.urdf.xacro (robot description, xacro)
@@ -61,4 +61,34 @@
         </collision>
     </link>
+    <!-- camera -->
+    <joint name='camera_joint' type='fixed'>
+        <origin xyz="0.41 0.0 0.15" />
+        <parent link="base_link" />
+        <child link="camera_link" />
+    </joint>
+    <!-- <origin xyz="0.4 0.0 0.21" /> -->
+    <link name="camera_link">
+        <visual name="camera_visual">
+            <origin xyz="0.0 0.0 0.0" />
+            <geometry>
+                <box size="0.02 0.25 0.06"/>
+            </geometry>
+            <material name="orange1">
+                <color rgba="1.0 0.5 0.2 1.0" />
+            </material>
+        </visual>
+        <collision>
+            <origin xyz="0.0 0.0 0.0" />
+            <geometry>
+               <box size="0.02 0.25 0.06"/>
+            </geometry>
+        </collision>
+    </link>
+    <joint name='camera_optical_joint' type='fixed'>
+        <origin xyz="0.0 0.0 0.0" rpy="0 0 0"/>
+        <parent link="camera_link" />
+        <child link="camera_link_optical" />
+    </joint>
+    <link name="camera_link_optical"/>
     <!-- Adding the tyres via xacro -->
      <!-- TOP RIGHT -->
