Commit message: added: added lidar to description and gazebo setup for lidar

File: parcbot_description/urdf/gazebo.xacro (robot description, xacro)
@@ -16,4 +16,33 @@
         <topic>cmd_vel</topic>
         </plugin>
+    </gazebo>
+    <!-- LIDAR -->
+    <gazebo reference="lidar_link">
+        <plugin filename="gz-sim-sensors-system" name="gz::sim::systems::Sensors">
+            <render_engine>ogre</render_engine>
+        </plugin>
+        <material>Gazebo/Green</material>
+        <sensor name="laser" type="gpu_lidar">
+            <pose> 0 0 0.043 0 0 0 </pose>
+            <visualize>true</visualize>
+            <update_rate>50</update_rate>
+            <always_on>true</always_on>
+            <ray>
+                <scan>
+                    <horizontal>
+                        <samples>360</samples>
+                        <min_angle>-1.57</min_angle>
+                        <max_angle>1.57</max_angle>
+                        <resolution>1</resolution>
+                    </horizontal>
+                </scan>
+                <range>
+                    <min>0.03</min>
+                    <max>12</max>
+                </range>
+            </ray>
+            <topic>/scan</topic>
+            <gz_frame_id>lidar_link</gz_frame_id>
+        </sensor>
     </gazebo>
     <!-- TYRES & CHASSIS -->

File: parcbot_description/urdf/parcbot.urdf.xacro (robot description, xacro)
@@ -11,4 +11,7 @@
     <material name="blue">
         <color rgba="0.3 0.0 1.0 1.0"/>
+    </material>
+    <material name="green">
+        <color rgba="0.1 1.0 0.0 1.0"/>
     </material>
     <link name="base_link">
@@ -32,4 +35,30 @@
         </inertial>
     </link>
+    <joint name="lidar_joint" type="fixed">
+        <origin xyz="0.0 0.0 0.225" rpy="0.0 0.0 0.0"/>
+        <parent link="base_link"/>
+        <child link="lidar_link"/>
+        <axis xyz="0.0 0.0 0.0"/>
+    </joint>
+    <link name="lidar_link">
+        <inertial>
+            <origin xyz="0.0 0.0 0.0" rpy="0.0 0.0 0.0"/>
+            <mass value="0.0"/>
+            <inertia ixx="0.0" ixy="0.0" ixz="0.0" iyy="0.0" iyz="0.0" izz="0.0"/>
+        </inertial>
+        <visual>
+            <origin xyz="0.0 0.0 0.075" rpy="0.0 0.0 0.0"/>
+            <geometry>
+                <cylinder radius="0.1" length="0.15"/>
+            </geometry>
+            <material name="green" />
+        </visual>
+        <collision>
+            <origin xyz="0.0 0.0 0.0" rpy="0.0 0.0 0.0"/>
+            <geometry>
+                <box size="0.0 0.0 0.0"/>
+            </geometry>
+        </collision>
+    </link>
     <!-- Adding the tyres via xacro -->
      <!-- TOP RIGHT -->

Commit message: feat: add camera sensor configuration to gazebo.xacro

File: parcbot_description/urdf/gazebo.xacro (robot description, xacro)
@@ -46,4 +46,31 @@
         </sensor>
     </gazebo>
+    <!-- CAMERA -->
+    <gazebo reference="camera_link_optical">
+        <material>Gazebo/Red</material>
+        <sensor type="camera" name="camera">
+            <update_rate>30.0</update_rate>
+            <camera name="head">
+                <camera_info_topic>camera/camera_info</camera_info_topic>
+                <horizontal_fov>1.3962634</horizontal_fov>
+                <image>
+                    <width>800</width>
+                    <height>600</height>
+                    <format>R8G8B8</format>
+                </image>
+                <clip>
+                    <near>0.02</near>
+                    <far>50</far>
+                </clip>
+                <!-- <noise>
+                    <type>gaussian</type>
+                    <mean>0.0</mean>
+                    <stddev>0.007</stddev>
+                </noise> -->
+            </camera>
+            <topic>camera/image_raw</topic>
+            <gz_frame_id>camera_link_optical</gz_frame_id>
+        </sensor>
+    </gazebo>
     <!-- TYRES & CHASSIS -->
     <!-- Chassis friction -->
